File: kicad/jack2bluetooth/jack2bluetooth.kicad_pcb (KiCad board)
At the start: 4 copper layers, 85.8 x 76 mm, 151 parts, among them IC1 TLV320AIC3101IRHBR, IC2 BQ25619RTWR, IC3 MCP23008T-E_SO, IC4 TPS62A01PDDCR, IC5 TPS62A01PDDCR, IC7 ESP32-WROVER-E-N16R8, J1 SJ3-35063A, J10 Conn_01x03_Pin, J2 USB_C_Receptacle, J3 Conn_01x03_Pin, J4 SJ1-2503A, J5 Conn_01x03_Pin, J6 Conn_01x04_Pin, J7 Conn_01x02_Pin, J8 Conn_01x02_Pin, J9 Conn_01x08_Pin, Q1 DMP3099L-13, Q2 BC846, Q3 BC846, SW1 SW_Push, SW2 SW_Push, SW3 SW_Push, SW4 SW_Push, SW5 SW_SPDT, SW6 SW_Push, SW7 SW_SPDT

Commit message: feat: generate gerber and bom
Changed lines of the file:
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@@
 			(pdf_back_fp_property_popups yes)
 			(pdf_metadata yes)
-			(pdf_single_document yes)
+			(pdf_single_document no)
 			(dxfpolygonmode yes)
 			(dxfimperialunits yes)
@@
 			(psnegative no)
 			(psa4output no)
-			(plot_black_and_white no)
+			(plot_black_and_white yes)
 			(sketchpadsonfab no)
 			(plotpadnumbers no)
@@
 			(crossoutdnponfab yes)
 			(subtractmaskfromsilk no)
-			(outputformat 4)
+			(outputformat 1)
 			(mirror no)
 			(drillshape 0)
 			(scaleselection 1)
-			(outputdirectory "../../doc/")
+			(outputdirectory "../../doc/gerber/")
 		)
 	)
@@
 		(tags "capacitor handsolder")
 		(property "Reference" "C7"
-			(at 0 -1.68 0)
+			(at -0.03 1.85 0)
 			(layer "F.SilkS")
 			(effects
@@
 		)
 		(fp_line
-			(start 9 15.7)
-			(end -9 15.7)
-			(stroke
-				(width 0.2)
-				(type solid)
-			)
-			(layer "F.SilkS")
-		)
-		(fp_line
 			(start 9 15.4)
 			(end 9 15.7)
@@
 			(layer "F.SilkS")
 		)
-		(fp_line
-			(start -9 -9)
-			(end -9 -15.7)
-			(stroke
-				(width 0.2)
-				(type solid)
-			)
-			(layer "F.SilkS")
-		)
-		(fp_line
-			(start -9 -15.7)
-			(end 9 -15.7)
-			(stroke
-				(width 0.2)
-				(type solid)
-			)
-			(layer "F.SilkS")
-		)
-		(fp_line
-			(start 9 -15.7)
-			(end 9 -9)
-			(stroke
-				(width 0.2)
-				(type solid)
-			)
-			(layer "F.SilkS")
-		)
 		(fp_arc
 			(start -10.1 -8.26)
@@
 		(tags "capacitor handsolder")
 		(property "Reference" "C12"
-			(at 0 -1.68 0)
+			(at -0.0125 1.675 0)
 			(layer "F.SilkS")
 			(effects
