File: kicad/jack2bluetooth/jack2bluetooth.kicad_sch (KiCad schematic)
At the start: 153 parts, among them IC1 TLV320AIC3101IRHBR, IC2 BQ25619RTWR, IC3 MCP23008T-E_SO, IC4 TPS62A01PDDCR, IC5 TPS62A01PDDCR, IC7 ESP32-WROVER-E-N16R8, J1 SJ3-35063A, J10 Conn_01x03_Pin, J2 USB_C_Receptacle, J3 Conn_01x03_Pin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

Commit message: feat: routing done, silkscreen done
Parts:
- removed TP2, TP6: TestPoint, TestPoint:TestPoint_Pad_D1.0mm, symbol Connector:TestPoint
Connections:
- net IO19: now also IC1.8 (SCL), IC2.5 (SCL), IC3.1 (SCL), J8.1 (Pin_1), TP11.1, TP28.1; no longer IC1.9 (SDA), IC2.6 (SDA), IC3.2 (SDA), J8.2 (Pin_2), TP12.1, TP29.1
- net IO21: now also IC1.9 (SDA), IC2.6 (SDA), IC3.2 (SDA), J8.2 (Pin_2), TP12.1, TP29.1; no longer IC1.8 (SCL), IC2.5 (SCL), IC3.1 (SCL), J8.1 (Pin_1), TP11.1, TP28.1
- net IO22: now also J9.5 (Pin_5); no longer J9.6 (Pin_6)
- net IO23: now also J9.6 (Pin_6); no longer J9.5 (Pin_5)
- net IO36: now also IC2.7 (/INT), R32.1, TP13.1; no longer IC3.8 (INT)
- net IO39: now also IC3.8 (INT); no longer IC2.7 (/INT), R32.1, TP13.1
- net POS1: now reaches JP1.1 (A), R10.2

Commit message: feat: generate gerber and bom
Parts:
- R11: value 10k -> 3k
- R4, R9: value 1k -> 3k
- R7, R8: value 1k -> 2k
Changed lines of the file:
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@@
 			)
 		)
-		(property "Value" "10k"
+		(property "Value" "3k"
 			(at 93.98 208.2799 0)
 			(effects
@@
 		(fields_autoplaced yes)
 		(property "Reference" "R8"
-			(at 273.685 107.9499 0)
+			(at 274.32 107.9499 0)
 			(effects
 				(font
@@
 			)
 		)
-		(property "Value" "1k"
-			(at 273.685 110.4899 0)
+		(property "Value" "2k"
+			(at 274.32 110.4899 0)
 			(effects
 				(font
@@
 			)
 		)
-		(property "Value" "1k"
+		(property "Value" "3k"
 			(at 236.22 102.8699 0)
 			(effects
@@
 			)
 		)
-		(property "Value" "1k"
+		(property "Value" "2k"
 			(at 256.54 111.7599 0)
 			(effects
@@
 		(fields_autoplaced yes)
 		(property "Reference" "R9"
-			(at 220.345 100.3299 0)
+			(at 220.98 100.3299 0)
 			(effects
 				(font
@@
 			)
 		)
-		(property "Value" "1k"
-			(at 220.345 102.8699 0)
+		(property "Value" "3k"
+			(at 220.98 102.8699 0)
 			(effects
 				(font
