File: kicad/jack2bluetooth/jack2bluetooth.kicad_sch (KiCad schematic)
At the start: 151 parts, among them IC1 TLV320AIC3101IRHBR, IC2 BQ25619RTWR, IC3 MCP23008T-E_SO, IC4 TPS62A01PDDCR, IC5 TPS62A01PDDCR, IC7 ESP32-WROVER-E-N16R8, J1 SJ3-35063A, J10 Conn_01x03_Pin, J2 USB_C_Receptacle, J3 Conn_01x03_Pin, J4 SJ1-2503A, J5 Conn_01x03_Pin, J6 Conn_01x04_Pin, J7 Conn_01x02_Pin, J8 Conn_01x02_Pin, J9 Conn_01x08_Pin, Q1 DMP3099L-13, Q2 BC846, Q3 BC846, SW1 SW_Push, SW2 SW_Push, SW3 SW_Push, SW4 SW_Push, SW5 SW_SPDT, SW6 SW_Push, SW7 SW_SPDT

Commit message: feat: update gerber, bom and add datasheets
Parts:
- C34: value 1u -> 1uF
Changed lines of the file:
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@@
 	(title_block
 		(title "Jack2Bluetooth")
+		(date "2026-03-17")
 		(rev "3.1")
 		(comment 4 "Author : Paul Capgras")
@@
 		)
 		(instances
-			(project ""
+			(project "jack2bluetooth"
 				(path "/4b32d186-730c-41ef-8802-f29516455534"
 					(reference "IC2")
@@
 		)
 		(instances
-			(project ""
+			(project "jack2bluetooth"
 				(path "/4b32d186-730c-41ef-8802-f29516455534"
 					(reference "D3")
@@
 		)
 		(instances
-			(project ""
+			(project "jack2bluetooth"
 				(path "/4b32d186-730c-41ef-8802-f29516455534"
 					(reference "PS1")
@@
 		)
 		(instances
-			(project ""
+			(project "jack2bluetooth"
 				(path "/4b32d186-730c-41ef-8802-f29516455534"
 					(reference "J4")
@@
 		)
 		(instances
-			(project ""
+			(project "jack2bluetooth"
 				(path "/4b32d186-730c-41ef-8802-f29516455534"
 					(reference "IC3")
@@
 			)
 		)
-		(property "Value" "1u"
+		(property "Value" "1uF"
 			(at 161.29 53.975 0)
 			(effects
@@
 		)
 		(instances
-			(project ""
+			(project "jack2bluetooth"
 				(path "/4b32d186-730c-41ef-8802-f29516455534"
 					(reference "Q1")
@@
 		)
 		(instances
-			(project ""
+			(project "jack2bluetooth"
 				(path "/4b32d186-730c-41ef-8802-f29516455534"
 					(reference "IC7")
@@
 		)
 		(instances
-			(project ""
+			(project "jack2bluetooth"
 				(path "/4b32d186-730c-41ef-8802-f29516455534"
 					(reference "J1")
@@
 		)
 		(instances
-			(project ""
+			(project "jack2bluetooth"
 				(path "/4b32d186-730c-41ef-8802-f29516455534"
 					(reference "J8")
@@
 		)
 		(instances
-			(project ""
+			(project "jack2bluetooth"
 				(path "/4b32d186-730c-41ef-8802-f29516455534"
 					(reference "IC5")
@@
 		)
 		(instances
-			(project ""
+			(project "jack2bluetooth"
 				(path "/4b32d186-730c-41ef-8802-f29516455534"
 					(reference "IC4")
@@
 		)
 		(instances
-			(project ""
+			(project "jack2bluetooth"
 				(path "/4b32d186-730c-41ef-8802-f29516455534"
 					(reference "F1")
@@
 		)
 		(instances
-			(project ""
+			(project "jack2bluetooth"
 				(path "/4b32d186-730c-41ef-8802-f29516455534"
 					(reference "Q2")
@@
 		)
 		(instances
-			(project ""
+			(project "jack2bluetooth"
 				(path "/4b32d186-730c-41ef-8802-f29516455534"
 					(reference "D5")
@@
 		)
 		(instances
-			(project ""
+			(project "jack2bluetooth"
 				(path "/4b32d186-730c-41ef-8802-f29516455534"
 					(reference "IC1")
